File: mcu-100-modular.kicad_sch (KiCad schematic)
At the start: 0 parts

Commit message: feat(mcu-100): actualizar esquematico, pcb y configuracion modular de espadines
Parts:
- added J1, J2, J3, J4: Espadines_2x15_Macho, LUISMATERIALES:PinHeader_2x15_P2.54mm_Vertical, symbol LUISMATERIALES:Espadines_2x15_Macho
- added M1: Module-mcu-0.7, hellen-one-mcu-0.7:mcu, symbol mcu:Module-mcu-0.7
- added M2: Module-mega-mcu144-0.7, hellen-one-mega-mcu144-0.7:mega-mcu144, symbol mega-mcu144:Module-mega-mcu144-0.7
- added M4: Module:mega-mcu100/0.3, hellen-one-mega-mcu100-0.3:mega-mcu100, symbol mega-mcu100:Module{colon}mega-mcu100/0.3

Commit message: fix(bom): remover modulos extra M2 y M4 para eliminar duplicados de U105 en BOM
Parts:
- removed M2: Module-mega-mcu144-0.7, hellen-one-mega-mcu144-0.7:mega-mcu144, symbol mega-mcu144:Module-mega-mcu144-0.7
- removed M4: Module:mega-mcu100/0.3, hellen-one-mega-mcu100-0.3:mega-mcu100, symbol mega-mcu100:Module{colon}mega-mcu100/0.3

Commit message: feat(sch, pcb): actualizar modulo M1 a mega-mcu100-0.3 y ajustar posicion en PCB
Parts:
- removed M1: Module-mcu-0.7, hellen-one-mcu-0.7:mcu, symbol mcu:Module-mcu-0.7
- added M1: Module:mega-mcu100/0.3, hellen-one-mega-mcu100-0.3:mega-mcu100, symbol mega-mcu100:Module{colon}mega-mcu100/0.3
